Commit message: minor changes to rviz launch

File: orthopillar_robot_spawner_pkg/models/orthopillar/model.urdf (robot description, URDF)
Before this commit: robot orthopillar_lidar, 4 links, 3 joints
Links:
- link chassis: geometry collision box size=.4 .2 .1; collision sphere radius=.06
- link laser_link: geometry collision box size=0.05 0.05 0.041; collision cylinder length=0.029 radius=0.021

Commit message: Fixing urdf model

File: orthopillar_robot_spawner_pkg/models/orthopillar/model.urdf (robot description, URDF)
Before this commit: robot orthopillar, 3 links, 2 joints
Links:
- added link laser_link, mass 0.1; collision box size=0.05 0.05 0.041; collision cylinder length=0.029 radius=0.021
- link chassis: geometry collision box size=0.3 0.6 0.2; collision sphere radius=.05
- link left_wheel: mass 1 -> None
- link right_wheel: mass 1 -> None
Joints:
- added joint laser_joint: type fixed, parent chassis, child laser_link, origin xyz=0  0.15    0.3 rpy=0  0  1.5707, axis 0  0  0
- joint left_wheel_hinge: axis -1 0 0 -> 0  0   1; origin xyz=0 0 0.03 rpy=0 0 0 -> xyz=0.11999  0.16     0.09999 rpy=0      1.5707  1.5707
- joint right_wheel_hinge: axis -1 0 0 -> 0 0 1; origin xyz=0 0 -0.03 rpy=0 0 0 -> xyz=0.12 -0.16  0.1 rpy=0      1.5707  1.5707

Commit message: first commit

File: orthopillar_robot_spawner_pkg/models/orthopillar/model.urdf (robot description, URDF)
Before this commit: robot orthopillar, 4 links, 3 joints
Links:
- link laser_link: geometry collision box size=0.05 0.05 0.041; collision cylinder length=0.029 radius=0.021
